File: DC080041B/DC080041B.kicad_sch (KiCad schematic)
At the start: 53 parts, among them SW1 Left Dip Switches, SW3 Back Dip Switches, U1 74S112, U10 74LS00, U11 74LS04, U12 8255A, U13 74LS08, U14 74LS244, U15 74LS244, U16 74LS74, U17 74LS30, U18 74LS00, U19 8288, U2 74S00, U20 8088_Max_Mode, U21 74LS10, U22 74LS112, U23 74LS74, U24 74S74, U25 74S74, U26 74S64, U27 74S00, U28 74LS04, U29 74LS04, U3 74S51, U30 74LS08, U31 74LS74, U32 74LS175, U33 74LS00, U34 8259A, U35 74LS00, U36 74LS00, U37 8087, U38 74LS175, U4 74S74, U5 8237A-5, U6 74LS240, U7 74S04, U8 74LS125, U9 74LS74, X1 14.31818MHz

Commit message: added U39-42
Parts:
- added U39: 74LS00, symbol 74xx:74LS00
- added U40: 74LS244, symbol 74xx:74LS244
- added U41: 74LS395, symbol 74xx:74LS395
- added U42: 74LS373, symbol 74xx:74LS373
Connections:
- net 8288_~{MRDC}: now also U40.2 (I0a)
- new net: U39.1, U40.12 (O3a), U41.13 (Q2)
- new net: U39.3, U42.11 (LE)
- new net: U39.2, U40.18 (O0a)

Commit message: added power & tidyed schematics
Connections:
- net GND: now also U1.8 (GND), U10.7 (GND), U11.7 (GND), U13.7 (GND), U16.7 (GND), U17.7 (GND), U18.7 (GND), U2.7 (GND), U21.7 (GND), U22.8 (GND), U23.7 (GND), U24.7 (GND), U25.7 (GND), U26.7 (GND), U27.7 (GND), U28.7 (GND), U29.7 (GND), U3.7 (GND), U30.7 (GND), U31.7 (GND), U33.7 (GND), U35.7 (GND), U36.7 (GND), U39.7 (GND), U4.7 (GND), U7.7 (GND), U8.7 (GND), U9.7 (GND)
- net VCC: now also U1.16 (VCC), U10.14 (VCC), U11.14 (VCC), U13.14 (VCC), U16.14 (VCC), U17.14 (VCC), U18.14 (VCC), U2.14 (VCC), U21.14 (VCC), U22.16 (VCC), U23.14 (VCC), U24.14 (VCC), U25.14 (VCC), U26.14 (VCC), U27.14 (VCC), U28.14 (VCC), U29.14 (VCC), U3.14 (VCC), U30.14 (VCC), U31.14 (VCC), U33.14 (VCC), U35.14 (VCC), U36.14 (VCC), U39.14 (VCC), U4.14 (VCC), U7.14 (VCC), U8.14 (VCC), U9.14 (VCC)
Other:
- moved on the sheet: U10A, U10D, U10E, U11A, U11D, U11E, U11G, U13A, U13C, U13E, U16A, U16C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

Commit message: added more 8288 output circuitry
Parts:
- removed U18: 74LS00, symbol 74xx:74LS00
- added DL3: (no value), symbol sperry:ADL-100L
- added R101: 4.7K, Resistor_THT:R_Array_SIP5, symbol Device:R_Network04
- added R103: 4.7K, Resistor_THT:R_Array_SIP9, symbol Device:R_Network08
- added U18, U46: 74LS04, symbol 74xx:74LS04
- added U43: 74LS175, symbol 74xx:74LS175
- added U44: 74LS00, symbol 74xx:74LS00
- added U45: 74LS20, symbol 74xx:74LS20
- added U47: 74LS245, symbol 74xx:74LS245
- added U48: 8253, Package_DIP:DIP-24_W15.24mm, symbol Timer:8253
- added U49: 74LS10, symbol 74xx:74LS10
- added U50: 74LS02, symbol 74xx:74LS02
- added U51: 74LS32, symbol 74xx:74LS32
Connections:
- net 8288_~{AIOWC}: now also U40.6 (I2a)
- net 8288_~{AMWC}: now also U40.4 (I1a), R103.4 (R3), R103.6 (R5), U45.5
- net 8288_~{IORC}: now also U40.8 (I3a), U41.5 (P2), R103.3 (R2)
- net 8288_~{MRDC}: now also R103.5 (R4), U45.2
- net GND: now also U14.10 (GND), U15.10 (GND), U32.8 (GND), U38.8 (GND), U40.10 (GND), U41.8 (GND), U42.10 (GND), U18.7 (GND)
- net VCC: now also U14.20 (VCC), U15.20 (VCC), U32.16 (VCC), U38.16 (VCC), U40.20 (VCC), U41.16 (VCC), U42.20 (VCC), U6.20 (VCC), R101.1 (common), R103.1 (common), U18.14 (VCC)
- net at U41.10 (~{CP}): now also U40.5 (O2b)
- net at U39.1, U40.12 (O3a), U41.13 (Q2): now also U47.9 (A7)
- net at U15.1 (OEa): now also U15.19 (OEb)
- net L4_OUT: now reaches L4.2
- net L4_OUT: now also U43.9 (Cp)
- net 8288_~{MWTC}: now reaches U19.9 (~{MWTC})
- net at U39.2, U40.18 (O0a): now also U47.3 (A1)
- net 8088_~{TEST}: now reaches U20.23 (~{TEST})
- net 8088_~{TEST}: now also R103.2 (R1)
- net 8088_~{RQ}/~{GT1}: now reaches U20.30 (~{RQ}/~{GT1})
- net 8088_~{RQ}/~{GT1}: now also R103.7 (R6)
- net at U17.6, U6.2 (I0a): now also U35.3
- net 8237_HRQ: now reaches U5.10 (HRQ)
- net 8237_HRQ: now also U18.9
- net 8237_~{MEMR}: now reaches U5.3 (~{MEMR})
- net 8237_~{MEMR}: now also U45.4, U46.11, U47.17 (B1)
- net at U35.1: now also R101.4 (R3)
- net at U35.2: now also U18.8
- net at U14.1 (OEa): now also U14.19 (OEb)
- net at U40.14 (O2a): now also U47.7 (A5)
- net at U40.15 (I2b): now also U40.7 (O1b)
- net at U40.16 (O1a): now also U47.5 (A3)
- new net: DL3.1 (IN), U44.13, U45.6
- new net: U18.3, U45.1, U46.1, U47.15 (B3)
- new net: U48.15 (CLK1), U48.18 (CLK2), U48.9 (CLK0)
- new net 8253_~{RD}: U47.11 (B7), U48.22 (~{RD}), U49.4, U50.9, U51.2
- new net 8253_~{WR}: U47.13 (B5), U48.23 (~{WR}), U49.5
- no-connect marks 8 -> 13
Other:
- moved on the sheet: U35A, U37, U39A, U40, U41, U42

Commit message: further tracing around upper chips
Parts:
- added JP9: Jumper_3_Bridged12, symbol Jumper:Jumper_3_Bridged12
- added P6: Conn_02x20_Odd_Even, symbol Connector_Generic:Conn_02x20_Odd_Even
- added R104: 4.7K, Resistor_THT:R_Array_SIP9, symbol Device:R_Network08
- added R114: 1K, Resistor_THT:R_Array_SIP5, symbol Device:R_Network04
- added U52: 74LS27, symbol 74xx:74LS27
- added U53: 74LS30, symbol 74xx:74LS30
- added U54: 74LS240, symbol 74xx:74LS240
- added U55, U60: 74LS08, symbol 74xx:74LS08
- added U56: 74LS32, symbol 74xx:74LS32
- added U57: 74LS245, symbol 74xx:74LS245
- added U58: 74LS273, symbol 74xx:74LS273
- added U59: 74LS04, symbol 74xx:74LS04
Connections:
- net 8288_CEN: now also U35.10, U53.3
- net VCC: now also R104.1 (common), R114.1 (common)
- net 8255A_~{WR}: now reaches U12.36 (~{WR})
- net 8255A_~{WR}: now also R104.7 (R6), U56.9
- net at U32.11 (~{Q2}): now also U35.9, U49.1
- net at U28.1: now also U52.6
- new net: U53.1, U55.6
- new net: U53.11, U55.8
- new net: U53.12, U55.11
- new net: U53.2, U55.3
- new net: U53.4, U54.3 (O3b)
- new net: U53.5, U54.5 (O2b)
- new net: U53.6, U54.9 (O0b)
- new net: U53.8, U56.10, U57.19 (CE)
- new net: U56.8, U58.11 (Cp)
- new net JP9_1: JP9.1 (A), U59.4
- new net JP9_2: JP9.2 (C), U60.4
- new net P6_16: JP9.3 (B), P6.16 (Pin_16), R114.5 (R4), U54.17 (I3b), U59.3
Other:
- moved on the sheet: U10E, U11G, U12, U13E, U16C, U17B, U18G, U1C, U21D, U22C, U23C, U24C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

Commit message: further work done in multiple areas
Parts:
- added C22: 1nF, symbol Device:C_Small
- added P1: Conn_01x04, symbol Connector_Generic:Conn_01x04
- added R21: 10K, symbol Device:R_Small
- added R4: 1K, symbol Device:R_Small
- added U61, U62, U63: 74LS373, symbol 74xx:74LS373
- added U64: 74LS138, symbol 74xx:74LS138
Connections:
- net 8088_CLK_INV: now also U9.11 (C)
- net 8088_RESET: now also U6.16 (O1a)
- net 8288_AEN: no longer U19.6 (~{AEN}), U8.3
- net GND: now also C22.1, U61.10 (GND), U62.10 (GND), U63.10 (GND)
- net VCC: now also U31.12 (D), R21.1, R4.1, U61.20 (VCC), U62.20 (VCC), U63.20 (VCC)
- net 8259_~{CS}: now reaches U34.1 (~{CS})
- net 8259_~{CS}: now also U5.11 (~{CS}), U64.15 (O0)
- net 8259_INT: now reaches U34.17 (INT)
- net 8259_INT: now also U20.18 (INTR)
- net at U32.14 (~{Q3}): now also U30.4, U31.13 (~{R})
- net at U13.1: now also R4.2
- net at U13.2: now also U6.3 (O3b)
- net at U13.3: now also U9.12 (D)
- net 8259_READY: now reaches U5.6 (READY)
- net 8259_READY: now also U30.6
- net at U31.10 (~{S}): now also U25.4 (~{S}), U30.8
- net U49_6: now reaches U31.11 (C)
- net U49_6: now also U49.6
- net at U31.8 (~{Q}): now also U30.5
- net POWER_GOOD: now reaches U6.13 (I1b)
- net POWER_GOOD: now also C22.2, P1.4 (Pin_4), R21.2
- net at U6.17 (I3b): now also U6.7 (O1b)
- net U9B_Q: now reaches U6.4 (I1a)
- net U9B_Q: now also U9.9 (Q)
- new net -12V: P1.2 (Pin_2)
- new net -5V: P1.1 (Pin_1)
- new net 12V: P1.3 (Pin_3)
- new net 8288_~{AEN}: U19.6 (~{AEN}), U61.11 (LE), U62.11 (LE), U63.11 (LE), U8.3
- no-connect marks 13 -> 14
Other:
- moved on the sheet: U11A, U11D, U11E, U13A, U13C, U16A, U18A, U18C, U18E, U18F, U19, U21A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

Commit message: started tracing NMI circuit
Parts:
- added U65: 74LS08, symbol 74xx:74LS08
- added U66: 74S74, symbol 74xx:74LS74
Connections:
- net 8088_READY: now also U20.22 (READY)
- net 8088_RESET: now also U20.21 (RESET)
- net at U35.4: now also U21.6
- net at U35.5: now also U31.5 (Q)
- net at U35.6: now also U28.9
- net 8088_NMI: now reaches U28.8
- net 8088_NMI: now also U20.17 (NMI)
- net at U10.11: now also U10.1, U21.3
- net at U10.13: now also U28.12
- net SW3_2: now reaches R100.3 (R2), SW3.2, U14.15 (I2b)
- net SW3_2: now also U36.1
- net 8255A_PB5: now reaches U12.23 (PB5)
- net 8255A_PB5: now also U28.13
- net at U36.3: now also U21.4
- net ISA_IO_CH_CK: now reaches U10.2
- net ISA_IO_CH_CK: now also R101.3 (R2)
- net at U21.5: now also U65.6
Other:
- moved on the sheet: U10A, U10D, U21B, U28D, U28F, U31A, U35B, U36A

Commit message: keyboard connector added
Parts:
- removed U65: 74LS08, symbol 74xx:74LS08
- added P3: Keyboard, symbol Connector_Generic:Conn_01x07
- added U65: 74LS74, symbol 74xx:74LS74
- added U67: 74LS02, symbol 74xx:74LS02
- added U68: 74LS245, symbol 74xx:74LS245
Connections:
- net 8237_~{MEMR}: now also U18.1, U50.2, U65.3 (C), U68.1 (A->B)
- net GND: now also P3.4 (Pin_4), P3.7 (Pin_7)
- net VCC: now also U31.4 (~{S}), P3.5 (Pin_5)
- net at U11.8: now also U65.1 (~{R})
- net 8255A_PC7: now reaches U12.10 (PC7)
- net 8255A_PC7: now also U65.5 (Q)
- net 8253_D7: now reaches U31.2 (D)
- net 8253_D7: now also U48.1 (D7)
- net at U31.3 (C): now also U51.6
- net at U21.5: now also U65.4 (~{S}), U65.6 (~{Q})
- new net: U65.2 (D), U67.1
- new net KEY_CLK: P3.1 (Pin_1)
- new net KEY_DATA: P3.2 (Pin_2)
- new net KEY_RESET: P3.3 (Pin_3)
- no-connect marks 14 -> 15
Other:
- moved on the sheet: U11D, U18A, U31A, U50A, U51B

Commit message: more circuits found and added
Parts:
- removed U16: 74LS74, symbol 74xx:74LS74
- added U69: 74LS244, symbol 74xx:74LS244
- added U70: 27128, Package_DIP:DIP-28_W15.24mm, symbol Memory_EPROM:27128
- added U71: 2732, Package_DIP:DIP-28_W15.24mm, symbol sperry:2732
Connections:
- net 8253_~{WR}: now also U51.10, U51.5
- net GND: now also U44.7 (GND), U45.7 (GND), U46.7 (GND), U49.7 (GND), U50.7 (GND), U51.7 (GND), U52.7 (GND), U53.7 (GND), U55.7 (GND), U56.7 (GND), U59.7 (GND), U60.7 (GND), U65.7 (GND), U66.7 (GND), U67.7 (GND)
- net VCC: now also U17.11, U17.12, U17.4, U44.14 (VCC), U45.14 (VCC), U46.14 (VCC), U49.14 (VCC), U50.14 (VCC), U51.14 (VCC), U52.14 (VCC), U53.14 (VCC), U55.14 (VCC), U56.14 (VCC), U59.14 (VCC), U60.14 (VCC), U65.14 (VCC), U66.14 (VCC), U67.14 (VCC)
- net U2_8_CLK: now reaches U2.8, U7.1, U7.3
- net U2_8_CLK: now also U23.3 (C), U29.1, U32.9 (Cp), U66.3 (C)
- net at U66.2 (D): now also U17.8
- net 8088_~{S2}: now reaches U19.18 (~{S2}), U20.28 (~{S2})
- net 8088_~{S2}: now also U17.1
- net 8088_~{S0}: now reaches U19.19 (~{S0}), U20.26 (~{S0})
- net 8088_~{S0}: now also U17.3
- net 8088_~{S1}: now reaches U19.3 (~{S1}), U20.27 (~{S1})
- net 8088_~{S1}: now also U17.2
- net U64_10: now reaches U51.4
- net U64_10: now also U51.1, U64.10 (O5)
- net U3_2: now reaches U3.2
- net U3_2: now also R101.5 (R4)
- net 8088_~{LOCK}: now reaches U20.29 (~{LOCK})
- net 8088_~{LOCK}: now also U17.5
- net at U52.8: now also U64.6 (E3)
- net at U64.11 (O4): now also U51.9
- net 8253_~{CS}: now reaches U64.13 (O2)
- net 8253_~{CS}: now also U48.21 (~{CS})
- net EPROM_A8: now reaches U64.4 (E1)
- net EPROM_A8: now also U45.10, U69.18 (O0a), U70.25 (A8), U71.23 (A8)
Other:
- moved on the sheet: U13B, U23A, U29A, U2A, U45B, U51C, U52C, U64, U66A, U8D
