File: DC080041B/DC080041B.kicad_sch (KiCad schematic)
At the start: 149 parts, among them J1 Bus_ISA_8bit, J2 Bus_ISA_8bit, J3 Bus_ISA_8bit, J4 Bus_ISA_8bit, J5 Bus_ISA_8bit, J6 Bus_ISA_8bit, J7 Bus_ISA_8bit, P1 Conn_01x04, P3 Keyboard, P6 Conn_02x20_Odd_Even, SW1 Left Dip Switches, SW3 Back Dip Switches, U1 74S112, U10 74LS00, U100 74LS244, U101 74LS175, U102 74LS20, U103 74S08, U104 74LS30, U105 8250, U106 74LS245, U11 74LS04, U12 8255A, U13 74LS08, U14 74LS244, U15 74LS244, U16 74LS322, U17 74LS30, U18 74LS04, U19 8288, U2 74S00, U20 8088_Max_Mode, U21 74LS10, U22 74LS112, U23 74LS74, U24 74S74, U25 74S74, U26 74S64, U27 74S00, U28 74LS04, U29 74LS04, U3 74S51, U30 74LS08, U31 74LS74, U32 74LS175, U33 74LS00, U34 8259A, U35 74LS00, U36 74LS00, U37 8087, U38 74LS175, U39 74LS00, U4 74S74, U40 74LS244, U41 74LS395, U42 74LS373, U43 74LS175, U44 74LS00, U45 74LS20, U46 74LS04, U47 74LS245, U48 8253, U49 74LS10, U5 8237A-5, U50 74LS02, U51 74LS32, U52 74LS27, U53 74LS30, U54 74LS240, U55 74LS08, U56 74LS32, U57 74LS245, U58 74LS273, U59 74LS04, U6 74LS240, U60 74LS08, U61 74LS373, U62 74LS373, U63 74LS373, U64 74LS138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

Commit message: tidying up
Connections:
- net GND: now also U102.7 (GND), U103.7 (GND), U104.7 (GND), U75.7 (GND), U76.7 (GND), U96.8 (GND)
- net VCC: now also U102.14 (VCC), U103.14 (VCC), U104.14 (VCC), U75.14 (VCC), U76.14 (VCC), U96.16 (VCC)
Other:
- moved on the sheet: U101, U102A, U102B, U103C, U103D, U11A, U11E, U16, U18C, U18F, U22A, U25B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

Commit message: started to finalise existing circuits
Parts:
- added R5: 1K, symbol Device:R_Small
- added R9: 22R, symbol Device:R_Small
Connections:
- net EPROM_A12: now also U36.9
- net EPROM_A9: now also U50.8, U64.5 (E2)
- net ISA_D0: now also U68.3 (A1)
- net ISA_D1: now also U68.2 (A0)
- net ISA_D2: now also U68.4 (A2)
- net ISA_D3: now also U68.5 (A3)
- net ISA_D4: now also U68.6 (A4)
- net ISA_D5: now also U68.7 (A5)
- net ISA_D6: now also U68.8 (A6)
- net ISA_D7: now also U68.9 (A7)
- net P6_3: now also U51.13
- net PARITY_D: now also U13.9, U8.8
- net U60_11: now also U36.10
- net VCC: now also R5.2
- net U4_C: now reaches U7.6, U7.9
- net U4_C: now also U4.11 (C), U4.3 (C), U9.3 (C)
- net BANK_2_D: now reaches U90.14 (DOUT), U90.2 (DIN), U91.14 (DOUT), U91.2 (DIN)
- net BANK_2_D: now also U68.16 (B2), U77.13 (F)
- net 4164_~{WRITE}: now reaches U78.3 (~{WRITE}), U80.3 (~{WRITE}), U82.3 (~{WRITE}), U84.3 (~{WRITE}), U86.3 (~{WRITE}), U88.3 (~{WRITE}), U90.3 (~{WRITE}), U92.3 (~{WRITE}), U94.3 (~{WRITE})
- net 4164_~{WRITE}: now also U79.3 (~{WRITE}), U8.10, U81.3 (~{WRITE}), U83.3 (~{WRITE}), U85.3 (~{WRITE}), U87.3 (~{WRITE}), U89.3 (~{WRITE}), U91.3 (~{WRITE}), U93.3 (~{WRITE}), U95.3 (~{WRITE}), R9.2
- net BANK_1_D: now reaches U92.14 (DOUT), U92.2 (DIN), U93.14 (DOUT), U93.2 (DIN)
- net BANK_1_D: now also U68.18 (B0), U77.1 (G)
- net at U51.11: now also U50.3
- net at U51.12: now also U67.4
- net BANK_5_D: now reaches U84.14 (DOUT), U84.2 (DIN), U85.14 (DOUT), U85.2 (DIN)
- net BANK_5_D: now also U68.13 (B5), U77.10 (C)
- net U9_~{R}: now reaches U4.10 (~{S})
- net U9_~{R}: now also R7.1, U1.10 (~{S}), U1.11 (J), U1.12 (K), U1.14 (~{R}), U1.2 (K), U1.3 (J), U1.4 (~{S}), U4.4 (~{S}), U9.1 (~{R}), U9.10 (~{S}), U9.13 (~{R}), U9.4 (~{S})
- net at U4.13 (~{R}): now also U1.15 (~{R}), U4.1 (~{R})
- net U4B_Q: now reaches U4.9 (Q)
- net U4B_Q: now also U1.13 (C)
- net U66_PU: now reaches U66.1 (~{R})
- net U66_PU: now also U66.10 (~{S}), R5.1
- net BANK_7_D: now reaches U80.14 (DOUT), U80.2 (DIN), U81.14 (DOUT), U81.2 (DIN)
- net BANK_7_D: now also U68.11 (B7), U77.8 (A)
- net BANK_0_D: now reaches U94.14 (DOUT), U94.2 (DIN), U95.14 (DOUT), U95.2 (DIN)
- net BANK_0_D: now also U68.17 (B1), U77.2 (H)
- net BANK_3_D: now reaches U88.14 (DOUT), U88.2 (DIN), U89.14 (DOUT), U89.2 (DIN)
- net BANK_3_D: now also U68.15 (B3), U77.12 (E)
- net at U36.8: now also U67.5
- net at U50.5: now also U50.10
- net U50_1: now reaches U50.6
- net U50_1: now also U50.1
- net U6_O0b: now reaches U9.2 (D)
- net U6_O0b: now also U6.9 (O0b)
- net U9A_Q: now reaches U9.5 (Q)
- net U9A_Q: now also U6.8 (I3a)
- net BANK_4_D: now reaches U86.14 (DOUT), U86.2 (DIN), U87.14 (DOUT), U87.2 (DIN)
- net BANK_4_D: now also U68.14 (B4), U77.11 (D)
- net at U4.5 (Q): now also U4.12 (D)
- net U101_~{Q2}: now reaches U101.11 (~{Q2})
- net U101_~{Q2}: now also U67.6
- net BANK_6_D: now reaches U82.14 (DOUT), U82.2 (DIN), U83.14 (DOUT), U83.2 (DIN)
- net BANK_6_D: now also U68.12 (B6), U77.9 (B)
- net U77_EVEN: now reaches U77.5 (Even)
- net U77_EVEN: now also U8.9
- net U18_4: now reaches U18.4
- net U18_4: now also U18.13
- net at U18.12: now also R9.1
- removed net 4164_PARITY_D: U13.9, U8.9
Other:
- moved on the sheet: U18F, U36C, U50B, U51D, U66B, U67B, U77, U7C, U7D, U9A, X1

Commit message: various improvements
Parts:
- added R105: 8K, Resistor_THT:R_Array_SIP9, symbol Device:R_Network08
Connections:
- net 8259_~{CS}: now also U64.14 (O1)
- net EPROM_A10: now also U52.10
- net EPROM_A5: now also U64.1 (A0)
- net EPROM_A7: now also U52.9, U64.3 (A2)
- net VCC: now also R105.1 (common)
- net 8255A_PB4: now reaches U11.9
- net 8255A_PB4: now also U12.22 (PB4), R105.8 (R7)
- net U77_ODD: now reaches U67.2
- net U77_ODD: now also U77.6 (Odd)
- net EPROM_A6: now reaches U70.4 (A6)
- net EPROM_A6: now also U64.2 (A1)
Other:
- moved on the sheet: U101, U102A, U102B, U45B, U46F, U52C, U60D, U67D, U75B

Commit message: more tracing
Parts:
- added U107: 74LS38, symbol 74xx:74LS38
Connections:
- net 8253_~{WR}: now also U105.18 (~{WR})
- net 8259_~{CS}: no longer U5.11 (~{CS}), U64.15 (O0)
- net 8288_CEN: now also U32.11 (~{Q2}), U49.1
- net U30_8: now also U65.13 (~{R})
- net U6_O2a: now also U31.1 (~{R}), U32.1 (~{Mr})
- net VCC: now also U48.11 (G0), U48.14 (G1), U65.10 (~{S}), U65.12 (D), U78.1 (~{RFSH}), U79.1 (~{RFSH}), U80.1 (~{RFSH}), U81.1 (~{RFSH}), U82.1 (~{RFSH}), U83.1 (~{RFSH}), U84.1 (~{RFSH}), U85.1 (~{RFSH}), U86.1 (~{RFSH}), U87.1 (~{RFSH}), U88.1 (~{RFSH}), U89.1 (~{RFSH}), U90.1 (~{RFSH}), U91.1 (~{RFSH}), U92.1 (~{RFSH}), U93.1 (~{RFSH}), U94.1 (~{RFSH}), U95.1 (~{RFSH})
- net 8259_IR0: now reaches U34.18 (IR0)
- net 8259_IR0: now also U48.10 (OUT0)
- net at L7.2, U24.3 (C), U26.6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: now also U30.13
- net U44_11: now reaches U103.2, U103.5, U44.11
- net 8255A_PB1: now reaches U12.19 (PB1)
- net 8255A_PB1: now also U107.13
- net at U25.12 (D): now also U25.5 (Q), U26.11, U26.13
- net at U27.10: now also U27.11
- net U27_8: now reaches U27.8
- net U27_8: now also U35.9
- net U13_6: now reaches U13.6, U23.2 (D)
- net U13_6: now also U50.11
- net U23A_Q: now reaches U50.12
- net U23A_Q: now also U23.5 (Q)
- net at U50.13: now also U49.2
- net 8237_DREQ0: now reaches U5.19 (DREQ0)
- net 8237_DREQ0: now also U65.9 (Q)
- net 8259_OUT1: now reaches U65.11 (C)
- net 8259_OUT1: now also U48.13 (OUT1)
- net at U30.11: now also U49.13
- net 8253_OUT2: now reaches U48.17 (OUT2)
- net 8253_OUT2: now also U107.12
- net U96A_O2: no longer names the net of U103.1, U96.6 (O2)
- net U96A_O3: no longer names the net of U103.4, U96.7 (O3)
- new net 8237_~{CS}: U5.11 (~{CS}), U64.15 (O0)
- no-connect marks 18 -> 20
Other:
- moved on the sheet: L8, L9, R106A, R106C, U103A, U103B, U10A, U10D, U11D, U13B, U21B, U25B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

Commit message: combined circuits and added SW3 info
Connections:
- net DB1 is gone; now on net EPROM_D1: U5.29 (DB1), U97.3 (D0), U98.17 (B1)
- net DB2 is gone; now on net EPROM_D2: U5.28 (DB2), U97.17 (D6), U98.16 (B2)
- net EPROM_D0 is gone; now on net 8237_DB0: U101.4 (D0), U70.11 (D0)
- net EPROM_D3 is gone; now on net 8237_DB3: U101.12 (D2), U70.15 (D3)
- net EPROM_~{OE} is gone; now on net EPROM_~{CE}: U70.22 (~{OE}), U75.6
- net DB4: now also U70.16 (D4)
- net DB5: now also U70.17 (D5)
- net DB6: now also U70.18 (D6)
- net DB7: now also U70.19 (D7)
- net GND: now also U74.5 (E2)
- net at U74.1 (A0): now also U101.2 (Q0)
- net P6_11: now reaches U74.10 (O5)
- net P6_11: now also P6.11 (Pin_11)
- net P6_10: now reaches U74.11 (O4)
- net P6_10: now also P6.10 (Pin_10)
- net P6_9: now reaches U74.12 (O3)
- net P6_9: now also P6.9 (Pin_9)
- net P6_8: now reaches U74.13 (O2)
- net P6_8: now also P6.8 (Pin_8)
- net EPROM_2732_~{CE}: now reaches U74.14 (O1)
- net EPROM_2732_~{CE}: now also P6.7 (Pin_7), U71.18 (~{CE}), U71.20 (~{OE}/VPP)
- net at U74.2 (A1): now also U101.15 (Q3)
- net at U74.3 (A2): now also U101.7 (Q1)
- net at U74.4 (E1): now also U101.10 (Q2)
- net P6_13: now reaches U74.7 (O7)
- net P6_13: now also P6.13 (Pin_13)
- net P6_12: now reaches U74.9 (O6)
- net P6_12: now also P6.12 (Pin_12)
- net EPROM_~{CE}: now reaches U70.20 (~{CE})
- net U46_2: no longer names the net of U46.2, U75.13
- net U67_13: no longer names the net of U60.13, U67.13, U75.2
Other:
- note added: "SW3-1: On=Normal loading Off=Repeated hardware self-test SW3-2: On=Medium res monitor Off=High res monitor SW3-3: On=Normal operation Off=Disable advanced features SW3-4: On=non-XON/XOFF printer Off=XON/XOFF printer SW3-5: On=No memory check Off=Memory check SW3-6: On=8087@8MHz Off=8087@4MHz SW3-7: On=8087 NOT installed Off=8087 installed SW3-8: On=8088@8MHz Off=8088@4MHz"
- note removed: "Switch 7: 8087 Related?"
- moved on the sheet: DL3, JP10, JP9, R103, R104, R105, R111, R114, R20, U101, U102A, U102B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

Commit message: slowly completing more circuits
Parts:
- removed U33: 74LS00, symbol 74xx:74LS00
- added DL4: (no value), symbol sperry:ADL-100L
- added J8: DB25_Socket_MountingHoles, symbol Connector:DB25_Socket_MountingHoles
- added JP3, JP8: Jumper_3_Bridged12, symbol Jumper:Jumper_3_Bridged12
- added JP7: Jumper_3_Open, symbol Jumper:Jumper_3_Open
- added R109: 2.2K, Resistor_THT:R_Array_SIP5, symbol Device:R_Network04
- added U108: 74LS245, symbol 74xx:74LS245
- added U109: 74LS74, symbol 74xx:74LS74
- added U110: 74LS125, symbol 74xx:74LS125
- added U111: SN75188, Package_DIP:DIP-14_W7.62mm, symbol sperry:SN75188
- added U112: HD75154, symbol sperry:HD75154
- added X2: 7372.800KHz, symbol Device:Crystal
Connections:
- net EPROM_A1 is gone; now on net 8237_A1: U55.1, U70.9 (A1)
- net 8237_DB0: now also U12.34 (D0), U14.3 (O3b)
- net 8237_DB3: now also U12.31 (D3), U14.9 (O0b)
- net DB4: now also U12.30 (D4), U14.18 (O0a)
- net DB5: now also U12.29 (D5), U14.16 (O1a)
- net DB6: now also U12.28 (D6), U14.14 (O2a)
- net DB7: now also U12.27 (D7), U14.12 (O3a)
- net EPROM_A5: now also U100.16 (O1a)
- net EPROM_A6: now also U100.3 (O3b)
- net EPROM_A7: now also U100.18 (O0a)
- net EPROM_D1: now also U12.33 (D1), U14.5 (O2b)
- net EPROM_D2: now also U12.32 (D2), U14.7 (O1b)
- net GND: now also U47.10 (GND), U47.19 (CE), JP7.3 (B), U110.1, U110.13, U110.4
- net ISA_A17: now also U52.3
- net ISA_A18: now also U52.5
- net ISA_A19: now also U52.4
- net VCC: now also R109.1 (common), U109.1 (~{R}), U109.10 (~{S}), U109.13 (~{R}), U109.4 (~{S}), U112.15 (VCC_ALT), U112.16 (VCC), U112.3 (1T)
- net 8259_IR4: now reaches U34.22 (IR4)
- net 8259_IR4: now also U110.8
- net at U24.1 (~{R}): now also U36.11
- net 8255A_PA0: now reaches U15.12 (O3a)
- net 8255A_PA0: now also U12.4 (PA0)
- net 8255A_PA1: now reaches U15.14 (O2a)
- net 8255A_PA1: now also U12.3 (PA1)
- net 8255A_PA2: now reaches U15.16 (O1a)
- net 8255A_PA2: now also U12.2 (PA2)
- net 8255A_PA3: now reaches U15.18 (O0a)
- net 8255A_PA3: now also U12.1 (PA3)
- net 8255A_PA4: now reaches U15.3 (O3b)
- net 8255A_PA4: now also U12.40 (PA4)
- net 8255A_PA5: now reaches U15.5 (O2b)
- net 8255A_PA5: now also U12.39 (PA5)
- net 8255A_PA6: now reaches U15.7 (O1b)
- net 8255A_PA6: now also U12.38 (PA6)
- net 8255A_PA7: now reaches U15.9 (O0b)
- net 8255A_PA7: now also U12.37 (PA7)
- net at U59.1: now also U56.11
- net at U59.2: now also U99.1 (OEa)
- net U72_~{ER}: now reaches U72.11 (~{Er})
- net U72_~{ER}: now also U36.6
- net at U29.11, U35.11: now also U52.2
- net at U36.12: now also U38.14 (~{Q3})
- net at U36.13: now also U38.10 (Q2), U38.5 (D1)
- net U38_~{Q2}: now reaches U13.4
- net U38_~{Q2}: now also U38.11 (~{Q2})
- net U38_Q1: now reaches U13.5
- net U38_Q1: now also U38.7 (Q1)
- net U52_12: now reaches U52.12
- net U52_12: now also U23.1 (~{R}), U38.1 (~{Mr})
- net 8237_A0: now reaches U70.10 (A0)
- net 8237_A0: now also U100.9 (O0b), U5.32 (A0), U108.11 (B7)
- net EPROM_A4: now reaches U70.6 (A4)
- net EPROM_A4: now also U100.5 (O2b)
- net EPROM_A3: now reaches U70.7 (A3)
- net EPROM_A3: now also U100.14 (O2a)
- net 8237_A2: now reaches U70.8 (A2)
- net 8237_A2: now also U100.7 (O1b), U5.34 (A2), U108.13 (B5), U108.6 (A4)
- net MSM5832_2: now reaches R111.4 (R3)
- net MSM5832_2: now also U56.1
- net at U56.3: now also U56.12, DL4.1 (IN)
- net 8237_A1: now reaches U5.33 (A1)
- net 8237_A1: now also U100.12 (O3a), U108.8 (A6)
- net 8237_A5: now reaches U5.35 (A3)
- net 8237_A5: now also U5.38 (A5), U108.4 (A2)
- net 8237_A4: now reaches U5.37 (A4)
- net 8237_A4: now also U108.15 (B3)
- net 8237_A6: now reaches U5.39 (A6)
- net 8237_A6: now also U108.17 (B1)
- net 8237_A7: now reaches U5.40 (A7)
- net 8237_A7: now also U108.2 (A0)
- net at U56.13: now also DL4.4 (TAP5?)
- net at U38.12 (D2): now also U38.15 (Q3)
- net at U38.9 (Cp): now also U29.2
- net U47_A->B: now reaches U97.1 (OE)
- net U47_A->B: now also U47.1 (A->B), U108.1 (A->B), U108.19 (CE)
- net ISA_IO_READY: now reaches U30.10
- net ISA_IO_READY: now also U30.9
- net 8250_SIN: now reaches U105.10 (SIN)
- net 8250_SIN: now also U112.13 (1Y)
- net 8250_SOUT: now reaches U105.11 (SOUT)
- net 8250_SOUT: now also U110.12
- net 8250_XIN: now reaches U105.16 (XIN)
- net 8250_XIN: now also U109.9 (Q)
- net 8250_INTR: now reaches U105.30 (INTR)
- net 8250_INTR: now also U110.9
- net 8250_~{OUT2}: now reaches U105.31 (~{OUT2})
- net 8250_~{OUT2}: now also R109.5 (R4), U110.10
- net at U100.11 (I0b): now also U108.9 (A7)
- net at U100.13 (I1b): now also U108.7 (A5)
- net at U100.15 (I2b): now also U108.5 (A3)
- net at U100.17 (I3b): now also U108.3 (A1)
- net at U100.2 (I0a): now also U108.18 (B0)
- net at U100.4 (I1a): now also U108.16 (B2)
- net at U100.6 (I2a): now also U108.14 (B4)
- net at U100.8 (I3a): now also U108.12 (B6)
- new net: U109.2 (D), U109.6 (~{Q})
- new net: JP8.2 (C), U109.3 (C)
- new net: U109.11 (C), U109.5 (Q)
- new net: U111.10 (3B), U111.12 (4A), U111.5 (2B)
- new net: JP3.1 (A), U111.11 (4Y)
- new net: U110.11, U111.13 (4B)
- new net: JP7.1 (A), U110.2
- new net: JP8.1 (A), U110.6
- new net: JP8.3 (B), U110.3
- new net: U110.5, X2.2
- new net: U109.12 (D), U109.8 (~{Q})
- new net J8_2: J8.2, JP3.2 (C)
- new net J8_20: J8.20 (P20), U111.6 (2Y)
- new net J8_3: U112.4 (1A)
- new net J8_4: J8.4, U111.8 (3Y)
- no-connect marks 20 -> 22
Other:
- moved on the sheet: U29A, U30A, U36D, U38, U52A, U56A, U56D, U57, U58, U59A, U70, U71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

Commit message: tracing the RTC circuit
Parts:
- added R10: 5.6K, symbol Device:R_Small
- added U113: 74LS125, symbol 74xx:74LS125
- added U33: M58321, symbol sperry:M58321
- added X3: Crystal, symbol Device:Crystal
Connections:
- net POWER_GOOD: now also U33.1 (STOP)
- net U57_CE: now also U56.5
- net U58_Cp: no longer R111.9 (R8), U58.11 (Cp)
- net VCC: now also R10.1
- net at U57.14 (B4), U58.18 (D7): now also U113.6
- net M58321_WRITE: now reaches R111.2 (R1)
- net M58321_WRITE: now also U58.19 (Q7), U33.11 (WRITE)
- net M58321_ADW: now reaches R111.6 (R5)
- net M58321_ADW: now also U33.3 (ADW)
- net M58321_~{BUSY}: now reaches U56.2
- net M58321_~{BUSY}: now also R111.9 (R8), U58.11 (Cp), U33.9 (~{BUSY})
- net at U99.11 (I0b): now also U99.12 (O3a), U33.7 (D3)
- net at U99.13 (I1b): now also U99.14 (O2a), U33.6 (D2)
- net at U99.15 (I2b): now also U99.16 (O1a), U33.5 (D1)
- net at U99.17 (I3b): now also U99.18 (O0a), U33.4 (D0)
- net at U99.19 (OEb): now also U56.6, U113.4
- net at U99.2 (I0a): now also U58.2 (Q0)
- net at U99.4 (I1a): now also U58.5 (Q1)
- net at U99.6 (I2a): now also U58.6 (Q2)
- net at U99.8 (I3a): now also U58.9 (Q3)
- net MSM5832_2 renamed M58321_CS1
- net M58321_CS1: now also U33.2 (CS1)
- new net: U33.14 (XT), X3.1
- new net: U33.15 (XT), X3.2
- new net: R10.2, U113.5, U33.10 (READ)
- no-connect marks 22 -> 24
Other:
- moved on the sheet: U56B
