File: DC080041B/DC080041B.kicad_sch (KiCad schematic)
At the start: 168 parts, among them J1 Bus_ISA_8bit, J2 Bus_ISA_8bit, J3 Bus_ISA_8bit, J4 Bus_ISA_8bit, J5 Bus_ISA_8bit, J6 Bus_ISA_8bit, J7 Bus_ISA_8bit, J8 DB25_Socket_MountingHoles, P1 Conn_01x04, P3 Keyboard, P6 Conn_02x20_Odd_Even, SW1 Left Dip Switches, SW3 Back Dip Switches, U1 74S112, U10 74LS00, U100 74LS244, U101 74LS175, U102 74LS20, U103 74S08, U104 74LS30, U105 8250, U106 74LS245, U107 74LS38, U108 74LS245, U109 74LS74, U11 74LS04, U110 74LS125, U111 SN75188, U112 HD75154, U113 74LS125, U12 8255A, U13 74LS08, U14 74LS244, U15 74LS244, U16 74LS322, U17 74LS30, U18 74LS04, U19 8288, U2 74S00, U20 8088_Max_Mode, U21 74LS10, U22 74LS112, U23 74LS74, U24 74S74, U25 74S74, U26 74S64, U27 74S00, U28 74LS04, U29 74LS04, U3 74S51, U30 74LS08, U31 74LS74, U32 74LS175, U33 M58321, U34 8259A, U35 74LS00, U36 74LS00, U37 8087, U38 74LS175, U39 74LS00, U4 74S74, U40 74LS244, U41 74LS395, U42 74LS373, U43 74LS175, U44 74LS00, U45 74LS20, U46 74LS04, U47 74LS245, U48 8253, U49 74LS10, U5 8237A-5, U50 74LS02, U51 74LS32, U52 74LS27, U53 74LS30, U54 74LS240, U55 74LS08, U56 74LS32, U57 74LS245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

Commit message: power LED circuits
Parts:
- added P5: LED, symbol Connector_Generic:Conn_01x02
- added R15, R25: 120R, symbol Device:R_Small
- added SW2: Left Dip Switches, symbol Switch:SW_DIP_x08
Connections:
- net GND: now also U113.2
- net VCC: now also U107.10, U107.2, U107.5, R15.1, R25.1
- net 8255A_PB2: now reaches U107.1
- net 8255A_PB2: now also U113.1, U12.20 (PB2)
- net at U107.3: now also SW2.13, SW2.14, SW2.15, SW2.16
- net at U107.8: now also U107.6, P5.2 (Pin_2)
- net 8255A_PB3: now reaches U107.9
- net 8255A_PB3: now also U107.4, U12.21 (PB3)
- net 8255A_PC0: now reaches U12.14 (PC0)
- net 8255A_PC0: now also R105.6 (R5), SW2.1, SW2.5
- net 8255A_PC1: now reaches U12.15 (PC1)
- net 8255A_PC1: now also R105.2 (R1), SW2.2, SW2.6
- net 8255A_PC2: now reaches U12.16 (PC2)
- net 8255A_PC2: now also R105.3 (R2), SW2.3, SW2.7
- net 8255A_PC3: now reaches U12.17 (PC3)
- net 8255A_PC3: now also R105.7 (R6), SW2.4, SW2.8
- net at U113.3: now also SW2.12
- new net: P5.1 (Pin_1), R15.2, R25.2
- no-connect marks 24 -> 26
Other:
- moved on the sheet: R105, U107A, U107B, U107C, U113A

Commit message: battery circuit
Parts:
- added BT1: Battery, symbol Device:Battery
- added C10: 220nF 16V, symbol Device:C_Small
- added D5, D6: 1N4148, Diode_THT:D_DO-35_SOD27_P7.62mm_Horizontal, symbol Diode:1N4148
- added R16: 1.2K, symbol Device:R_Small
- added R17: 380R, symbol Device:R_Small
- P5: footprint (none) -> Connector_JST:JST_XH_B2B-XH-A_1x02_P2.50mm_Vertical
Connections:
- net 12V: now also R16.1
- net 8255A_PB5: now also R105.4 (R3)
- net GND: now also BT1.2 (-), C10.2
- net VCC: now also D5.1 (K)
- net at U33.16 (VCC): now also C10.1, D6.1 (K), R17.1
- new net: BT1.1 (+), R17.2
- new net: D5.2 (A), D6.2 (A), R16.2
Other:
- moved on the sheet: DL4, JP10, JP3, JP7, JP8, JP9, P5, R10, R103, R104, R109, R111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

Commit message: speaker circuit
Parts:
- removed C10: 220nF 16V, symbol Device:C_Small
- added C10: 220nF 16V, symbol Device:C_Polarized_Small
- added C5: 220uF 10V, symbol Device:C_Polarized_Small
- added D1: 1N4148, Diode_THT:D_DO-35_SOD27_P7.62mm_Horizontal, symbol Diode:1N4148
- added P4: Speaker, symbol Connector_Generic:Conn_01x02
- added R11, R12: 560R, symbol Device:R_Small
- added R22: 10R, symbol Device:R_Small
- added R23, R24: 100R, symbol Device:R_Small
- added TR1: C2320, symbol Simulation_SPICE:NPN
Connections:
- net 8255A_PA0: now also U16.13 (H/Qh)
- net 8255A_PA1: now also U16.7 (G/Qg)
- net 8255A_PA2: now also U16.14 (F/Qf)
- net 8255A_PA3: now also U16.6 (E/Qe)
- net 8255A_PA4: now also U16.15 (D/Qd)
- net 8255A_PA5: now also U16.5 (C/Qc)
- net 8255A_PA6: now also U16.16 (B/Qb)
- net 8255A_PA7: now also U16.4 (A/Qa)
- net GND: now also C10.2, D1.2 (A), P4.2 (Pin_2), TR1.3 (E)
- net KEY_RESET: now also U43.1 (~{Mr})
- net VCC: now also U16.18 (SE), U16.19 (DS), U16.2 (S/P), U16.20 (VCC), U16.3 (D0), R11.1, R23.2, R24.2
- net at D6.1 (K), R17.1, U33.16 (VCC): now also C10.1
- net 8255A_PB7: now reaches U12.25 (PB7)
- net 8255A_PB7: now also U11.11, U16.8 (OE)
- net at U113.11: now also U43.5 (D1)
- net at U66.11 (C): now also U16.11 (Clk), U43.3 (~{Q0})
- net at U66.12 (D): now also U16.12 (Qh)
- net at U66.8 (~{Q}): now also U113.10
- net at U66.9 (Q): now also U16.1 (G)
- net at U16.17 (D1): now also U113.8
- net 8253_CLK: now reaches U48.15 (CLK1), U48.18 (CLK2), U48.9 (CLK0)
- net 8253_CLK: now also U43.10 (Q2)
- net at U107.11: now also R11.2, R12.1
- new net: C5.1, P4.1 (Pin_1)
- new net: C5.2, R22.2, R23.1, R24.1
- new net: R22.1, TR1.1 (C)
- new net: D1.1 (K), R12.2, TR1.2 (B)
Other:
- note added: "Battery"
- note added: "Speaker Control"
- moved on the sheet: BT1, D5, D6, R16, R17, U107D, U113C, U113D, U11E, U16, U43, U66B

Commit message: tidying and miniturising circuits
Parts:
- SW2: value Left Dip Switches -> Right Dip Switches
Connections:
- net GND: now also U69.10 (GND), U97.10 (GND), U98.10 (GND)
- net VCC: now also U69.20 (VCC), U97.20 (VCC), U98.20 (VCC)
Other:
- note added: "SW2 / Right Dip Switches"
- moved on the sheet: P5, R105, R15, R25, SW2, U107A, U107B, U107C, U113A, U53A, U54, U55A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

Commit message: optocoupler traced
Parts:
- added D7: 1N4148, Diode_THT:D_DO-35_SOD27_P7.62mm_Horizontal, symbol Diode:1N4148
- added NF8: 470pF, symbol Device:C_Feedthrough
- added R1: 4.6K, symbol Device:R_Small
- added R18: 120K, symbol Device:R_Small
- added R19: 47R, symbol Device:R_Small
- added U114: PS2001, Package_DIP:DIP-6_W7.62mm, symbol Isolator:4N35
Connections:
- net 8237_DB0 is gone; now on net EPROM_D0: U101.4 (D0), U12.34 (D0), U14.3 (O3b), U5.30 (DB0), U70.11 (D0), U72.15 (D1), U97.18 (D7), U98.18 (B0)
- net 8237_DB3 is gone; now on net EPROM_D3: U101.12 (D2), U12.31 (D3), U14.9 (O0b), U5.27 (DB3), U70.15 (D3), U72.3 (D4), U97.4 (D1), U98.15 (B3)
- net 8253_D7 is gone; now on net DB7: U31.2 (D), U48.1 (D7)
- net 8288_CEN is gone; now on net 8237_~{MEMR}: U19.15 (CEN), U21.9, U32.11 (~{Q2}), U35.10, U49.1, U53.3
- net 8288_~{AIOWC} is gone; now on net 8237_~{MEMR}: U19.12 (~{AIOWC}), U27.5, U34.2 (~{WR}), U40.6 (I2a)
- net ISA_A19 is gone; now on net 8237_~{MEMR}: J1.43 (BA19), J2.43 (BA19), J3.43 (BA19), J4.43 (BA19), J5.43 (BA19), J6.43 (BA19), J7.43 (BA19), U102.5, U52.4
- net 8237_A0: now also U48.19 (A0), U72.14 (Wa)
- net 8237_A1: now also U48.20 (A1), U72.13 (Wb)
- net 8237_~{MEMR}: now also U26.9, U28.1, U30.1, U31.9 (Q), U32.13 (D3), U32.15 (Q3), U44.4, U52.6, U96.13 (A1), U96.3 (A1)
- net 8288_~{AMWC}: now also U41.6 (P3)
- net DB4: now also U48.4 (D4)
- net DB5: now also U48.3 (D5)
- net DB6: now also U48.2 (D6)
- net EPROM_D1: now also U48.7 (D1), U72.1 (D2)
- net EPROM_D2: now also U48.6 (D2), U72.2 (D3)
- net GND: now also U113.12, U113.9, NF8.2, R18.2, U114.4
- net ISA_A17: now also U72.9 (Q2)
- net ISA_A18: now also U72.7 (Q3)
- net ISA_D3: now also U72.6 (Q4)
- net VCC: now also U41.1 (~{MR}), U41.7 (LD/~{SH}), R1.1
- net at U41.12 (Q3): now also U40.14 (O2a), U47.7 (A5)
- net U49_12: now reaches U41.9 (~{OE})
- net U49_12: now also U49.12
- net ISA_TC: now reaches J5.27 (TC)
- net ISA_TC: now also J1.27 (TC), J2.27 (TC), J3.27 (TC), J4.27 (TC), J6.27 (TC), J7.27 (TC), U18.6
- net 8255A_PB0: now reaches U12.18 (PB0)
- net 8255A_PB0: now also U48.16 (G2)
- net 8255A_PB6: now reaches U12.24 (PB6)
- net 8255A_PB6: now also U113.13
- net 8237_DACK2: now reaches U72.4 (Rb)
- net 8237_DACK2: now also U5.14 (DACK2)
- net 8237_DACK3: now reaches U72.5 (Ra)
- net 8237_DACK3: now also U5.15 (DACK3)
- net J8_18: now reaches J8.18 (P18)
- net J8_18: now also NF8.1
- net J8_25: now reaches J8.25 (P25)
- net J8_25: now also D7.2 (A), U114.2
- net 8237_~{EOP}: now reaches U5.36 (~{EOP})
- net 8237_~{EOP}: now also U18.5
- net at U11.1: now also R1.2, U114.5
- net EPROM_D3: now reaches U48.5 (D3)
- net EPROM_D0: now reaches U48.8 (D0)
- new net: R18.1, U114.6
- new net: D7.1 (K), R19.2, U114.1
- new net: NF8.3, R19.1
- no-connect marks 26 -> 29
Other:
- moved on the sheet: U11A, U18C, U39B, U52B, U52C

Commit message: serial port + moved component fix
Parts:
- added JP1, JP2: Jumper_3_Bridged12, symbol Jumper:Jumper_3_Bridged12
- added U115: HD75154, symbol sperry:HD75154
Connections:
- net J8_3 is gone; now on an unnamed net: U112.4 (1A)
- net 8237_~{MEMR}: no longer J1.43 (BA19), J2.43 (BA19), J3.43 (BA19), J4.43 (BA19), J5.43 (BA19), J6.43 (BA19), J7.43 (BA19), U102.5, U19.12 (~{AIOWC}), U19.15 (CEN), U21.9, U26.9, U27.5, U28.1, U30.1, U31.9 (Q), U32.11 (~{Q2}), U32.13 (D3), U32.15 (Q3), U34.2 (~{WR}), U35.10, U40.6 (I2a), U44.4, U49.1, U52.4, U52.6, U53.3, U96.13 (A1), U96.3 (A1)
- net GND: now also J8.7, J8.SH (PAD)
- net at J8.11: now also JP1.2 (C)
- net at J8.13: now also J8.3
- net at J8.22 (P22): now also U115.4 (1A)
- net at J8.5: now also U115.7 (4A)
- net at J8.6: now also U115.6 (3A)
- net at J8.8: now also U115.5 (2A)
- net at J8.9: now also JP2.2 (C)
- net J8_18: no longer names the net of J8.18 (P18), NF8.1
- net J8_2: no longer names the net of J8.2, JP3.2 (C)
- net J8_20: no longer names the net of J8.20 (P20), U111.6 (2Y)
- net J8_25: no longer names the net of D7.2 (A), J8.25 (P25), U114.2
- net J8_4: no longer names the net of J8.4, U111.8 (3Y)
- new net: U28.1, U44.4, U52.6, U96.13 (A1), U96.3 (A1)
- new net: U26.9, U31.9 (Q), U32.13 (D3)
- new net: U32.11 (~{Q2}), U49.1
- new net: U30.1, U32.15 (Q3)
- new net 8288_CEN: U19.15 (CEN), U21.9, U35.10, U53.3
- new net 8288_~{AIOWC}: U19.12 (~{AIOWC}), U27.5, U34.2 (~{WR}), U40.6 (I2a)
- new net ISA_A19: J1.43 (BA19), J2.43 (BA19), J3.43 (BA19), J4.43 (BA19), J5.43 (BA19), J6.43 (BA19), J7.43 (BA19), U102.5, U52.4
Other:
- moved on the sheet: D7, J8, JP3, JP7, JP8, NF8, R1, R18, R19, U109A, U109B, U110A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
