File: DC280182B_FDC/DC280182B_FDC.kicad_sch (KiCad schematic)
At the start: 0 parts

Commit message: clock circuit
Parts:
- added C05: 10nF 50V, symbol Device:C_Small
- added R15: 680K, symbol Device:R_Small
- added U2: SED9420C, Package_DIP:DIP-24_18.0mmx34.29mm_W15.24mm_LongPads, symbol sperry:SED9420C
- added U24: 74LS14, symbol 74xx:74LS14
- added X01: 16MHz, symbol Device:Crystal
Connections:
- new net: C05.2, R15.1, U2.1 (OSC1)
- new net: R15.2, U2.2 (OSC2)
- new net: C05.1, U24.2
- new net: U24.1, X01.2

Commit message: added all chips & layed basic traces
Parts:
- added RN1: R_Network04, Resistor_THT:R_Array_SIP5, symbol Device:R_Network04
- added SW01: SW_DIP_x04, symbol Switch:SW_DIP_x04
- added U10: 74LS153, symbol 74xx:74LS153
- added U11, U17: 74LS08, symbol 74xx:74LS08
- added U12, U14: 74LS175, symbol 74xx:74LS175
- added U13: 74LS74, symbol 74xx:74LS74
- added U15: 74LS00, symbol 74xx:74LS00
- added U16: 74LS04, symbol 74xx:74LS04
- added U18: 74LS125, symbol 74xx:74LS125
- added U19, U27, U28, U8, U9: 7438, symbol 74xx_IEEE:7438
- added U20: 4016, symbol 4xxx:4016
- added U21: 74LS393, symbol 74xx:74LS393
- added U22, U3, U7: 74LS240, symbol 74xx:74LS240
- added U23, U5, U6: 74LS32, symbol 74xx:74LS32
- added U24: 74LS14, symbol 74xx:74LS14
- added U25: 74LS30, symbol 74xx:74LS30
- added U26: 74LS02, symbol 74xx:74LS02
- added U29: 74LS273, symbol 74xx:74LS273
- added U30: 74LS245, symbol 74xx:74LS245
- added U4: 74LS10, symbol 74xx:74LS10
Connections:
- net at U24.9: now also U16.1, U4.2, U4.3
- net at U24.12: now also U16.3, U4.5
- new net: U9.12, U9.13
- new net: U5.10, U5.13
- new net: RN1.5 (R4), SW01.4, U22.11 (I0b)
- new net: RN1.4 (R3), SW01.3, U22.13 (I1b)
- new net: RN1.3 (R2), SW01.2, U22.15 (I2b)
- new net: RN1.2 (R1), SW01.1, U22.17 (I3b)
- new net: U18.4, U22.19 (OEb)
- new net: U16.4, U4.1
- new net: U25.3, U26.1
- new net: U17.8, U6.2, U6.6
- new net: U17.5, U24.6
- new net: U18.10, U18.13
- new net: U23.3, U23.4
- new net: U6.12, U6.8
- new net: U11.1, U11.2
- new net: U5.1, U5.4
- new net: U19.10, U19.12, U19.13, U19.9
- new net: U8.1, U8.2
- new net: U12.10 (Q2), U12.13 (D3)
- new net: U12.2 (Q0), U12.5 (D1)
- new net: U8.4, U8.5
- new net: U11.12, U11.13
- new net: U8.10, U8.9
- new net GND: SW01.5, SW01.6, SW01.7, SW01.8, U22.1 (OEa)
- new net VCC: RN1.1 (common), U13.10 (~{S})
- no-connect marks 0 -> 14
Other:
- moved on the sheet: U24D, U24F, U24G

Commit message: various touch ups
Parts:
- added BF01, BF06, BF08, BF09, BF10, BF11, BF12, BF13, BF7: L_Small, symbol Device:L_Small
- added D01: D_Small, symbol Device:D_Small
- added J1: Bus_ISA_8bit, symbol Connector:Bus_ISA_8bit
- added JP01: Jumper_3_Bridged12, symbol Jumper:Jumper_3_Bridged12
- added P121: Internal Floppy Connector, symbol Connector_Generic:Conn_02x17_Odd_Even
- added R1, R12: 4.7K, symbol Device:R_Small
- added R10: 150R, symbol Device:R_Small
- added R11: 3.3K, symbol Device:R_Small
- added R18: 560K, symbol Device:R_Small
- added R19: 180R, symbol Device:R_Small
- added R20: 1.8K, symbol Device:R_Small
- added U1: D765AC, Package_DIP:DIP-40_W15.24mm, symbol sperry:D765AC
Connections:
- net GND: now also U10.1 (Ea), U10.3 (I3a), U10.8 (GND), U20.5, U20.6, U30.10 (GND), U30.19 (CE), P121.1 (Pin_1), P121.11 (Pin_11), P121.13 (Pin_13), P121.15 (Pin_15), P121.17 (Pin_17), P121.19 (Pin_19), P121.21 (Pin_21), P121.23 (Pin_23), P121.25 (Pin_25), P121.27 (Pin_27), P121.29 (Pin_29), P121.3 (Pin_3), P121.31 (Pin_31), P121.33 (Pin_33), P121.5 (Pin_5), P121.7 (Pin_7), P121.9 (Pin_9)
- net VCC: now also R1.1, R10.1
- net at U5.10, U5.13: now also U6.6
- net U5_8: now reaches U5.8
- net U5_8: now also U29.11 (Cp)
- net at U28.10: now also U28.9
- net at U14.1 (~{Mr}): now also U11.3, U19.10, U19.12, U19.13, U19.9
- net at U24.8: now also U16.1
- net at U4.2, U4.3: no longer U16.1, U24.9
- net at U3.12 (O3a): now also U7.18 (O0a), JP01.3 (B)
- net at U3.14 (O2a): now also U7.5 (O2b), BF01.1
- net at U3.17 (I3b): now also U6.3
- net at U3.18 (O0a): now also U11.9, U7.7 (O1b)
- net NREADDATA: now reaches U3.6 (I2a)
- net NREADDATA: now also P121.30 (Pin_30), R10.2
- net at U9.1: now also U11.11, U8.10, U8.9, U9.2
- net at U18.5: now also JP01.2 (C)
- net at U20.10: now also R11.2
- net at U20.11: now also R12.2
- net at U20.12: now also U20.13
- net at U23.11: now also U28.12, U28.13
- net at U4.9: now also U4.13
- net at U16.12: now also U18.10, U18.13
- net at U16.13: now also U29.12 (Q4)
- net D765AC_~{DACK}: now reaches U15.6
- net D765AC_~{DACK}: now also U12.1 (~{Mr})
- net at U17.10: now also U25.8
- net at U17.8, U6.2: now also U6.5; no longer U6.6
- net at U2.16 (LPF1): now also R19.1
- net at U2.6 (SYNC): now also R18.2
- net at U2.7 (R_DATA): now also BF01.2
- net at U13.13 (~{R}): now also U13.1 (~{R}), U24.4, U29.1 (~{Mr})
- net at U13.9 (Q): now also U23.1, U23.4
- net ISA_DRQ2: now reaches U18.11
- net at U18.12: now also U12.15 (Q3)
- net at U9.10: now also U9.9
- net at U23.3: no longer U23.4
- net at U28.4: now also U28.5
- net at U6.13: now also U30.1 (A->B)
- net at U4.12: now also U5.2
- net at U28.1: now also U28.2
- net ISA_A29: now reaches U24.13
- net ISA_A29: now also J1.60 (BA02)
- net at U8.12: now also U8.13
- net at U29.13 (D4): now also BF10.2
- net at U29.14 (D5): now also BF08.2
- net at U29.17 (D6): now also BF06.2
- net at U29.18 (D7): now also BF7.2
- net at U29.3 (D0): now also BF13.2
- net at U29.4 (D1): now also BF09.2
- net at U29.7 (D2): now also BF11.2
- net at U29.8 (D3): now also BF12.2
- net at U12.12 (D2): now also U12.7 (Q1)
- net D765AC_DRQ: now reaches U12.4 (D0)
- net at U12.9 (Cp): now also U21.9 (Q2)
- net at U10.10 (I0b): now also U10.11 (I1b), U10.12 (I2b), U10.13 (I3b)
- net at U9.4: now also U9.5
- net at U30.11 (B7): now also BF13.1
- net at U30.12 (B6): now also BF12.1
- net at U30.13 (B5): now also BF09.1
- net at U30.14 (B4): now also BF11.1
- net at U30.15 (B3): now also BF10.1
- net at U30.16 (B2): now also BF08.1
- net at U30.17 (B1): now also BF7.1
- net at U30.18 (B0): now also BF06.1
- net ISA_A2: now reaches U30.2 (A0)
- net ISA_A3: now reaches U30.3 (A1)
- net ISA_A4: now reaches U30.4 (A2)
- net ISA_A6: now reaches U30.5 (A3)
- net ISA_A7: now reaches U30.6 (A4)
- net ISA_A5: now reaches U30.7 (A5)
- net ISA_A8: now reaches U30.8 (A6)
- net ISA_A9: now reaches U30.9 (A7)
- net ISA_RESET: now reaches U24.3
- net ISA_RESET: now also J1.2 (RESET)
- new net: R19.2, R20.1
- new net: D01.1 (K), R18.1
- new net: JP01.1 (A), R1.2
- new net DB0: U1.6 (DB0)
- new net DB1: U1.7 (DB1)
- new net DB2: U1.8 (DB2)
- new net DB3: U1.9 (DB3)
- new net DB4: U1.10 (DB4)
- new net DB5: U1.11 (DB5)
- new net DB6: U1.12 (DB6)
- new net DB7: U1.13 (DB7)
- no-connect marks 14 -> 12
Other:
- note added: "CHECK THIS"
- moved on the sheet: C05, R15, RN1, SW01, U11A, U11C, U11D, U12, U13A, U13B, U14, U15B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
